Commit message: mobile robot old version

File: src/mobile_robot_v1/urdf/gazebo_control.xacro (robot description, xacro)
@@ -6,5 +6,5 @@
             <left_joint>left_wheel_joint</left_joint>
             <right_joint>right_wheel_joint</right_joint>
-            <wheel_separation>0.3</wheel_separation>
+            <wheel_separation>0.35</wheel_separation>
             <wheel_diameter>0.1</wheel_diameter>
             <!-- Limits-->

File: src/mobile_robot_v1/urdf/robot_core.xacro (robot description, xacro)
@@ -14,21 +14,21 @@
     </material>
     <!--Define inertial property macro -->
-    <xacro:macro name="box_inertial" params="m w d h">
+    <xacro:macro name="box_inertial" params="m w d h *origin">
         <inertial>
-            <origin xyz="0.15 0.0 0.75" rpy="0.0 0.0 0.0"/>
+            <xacro:insert_block name="origin"/>
             <mass value="${m}"/>
             <inertia ixx="${(m/12) * (h*h + d*d)}" ixy="0.0" ixz="0.0" iyy="${(m/12) * (w*w + h*h)}" iyz="0.0" izz="${(m/12) * (w*w + d*d)}"/>
         </inertial>
     </xacro:macro>
-    <xacro:macro name="cylinder_inertia" params="m r h">
+    <xacro:macro name="cylinder_inertia" params="m r h *origin">
         <inertial>
-            <origin xyz="0.0 0.0 0.0" rpy="0.0 0.0 0.0"/>
+            <xacro:insert_block name="origin"/>
             <mass value="${m}"/>
             <inertia ixx="${(m/12) * (3*r*r + h*h)}" ixy="0.0" ixz="0.0" iyy="${(m/12) * (3*r*r + h*h)}" iyz="0.0" izz="${(m/2) * (r * r)}"/>
         </inertial>
     </xacro:macro>
-    <xacro:macro name="sphere_inertia" params="m r">
+    <xacro:macro name="sphere_inertia" params="m r *origin">
         <inertial>
-            <origin xyz="0.0 0.0 0.0" rpy="0.0 0.0 0.0"/>
+            <xacro:insert_block name="origin"/>
             <mass value="${m}"/>
             <inertia ixx="${(2/5) * m * (r*r)}" ixy="0.0" ixz="0.0" iyy="${(2/5) * m * (r*r)}" iyz="0.0" izz="${(2/5) * m * (r*r)}"/>
@@ -45,5 +45,5 @@
             </geometry>
             <material name="white" />
-            <origin xyz="0.15 0.0 0.075" rpy="0.0 0.0 0.0"/>
+            <origin xyz="0.15 0.0 0.075" />
         </visual>
         <collision>
@@ -53,5 +53,7 @@
             <origin xyz="0.15 0.0 0.075" rpy="0.0 0.0 0.0"/>
         </collision>
-        <xacro:box_inertial m="0.5" w="0.3" d="0.3" h="0.15"/>
+        <xacro:box_inertial m="0.5" w="0.3" d="0.3" h="0.15">
+            <origin xyz="0.15 0.0 0.75" rpy="0.0 0.0 0.0"/>
+        </xacro:box_inertial>
     </link>
     <gazebo reference="chassis">
@@ -61,5 +63,5 @@
         <parent link="base_link"/>
         <child link="chassis"/>
-        <origin xyz="-0.1 0.0 0.0" rpy="0.0 0.0 0.0"/>
+        <origin xyz="-0.1 0.0 0.0" />
     </joint>
     <!--left wheel link-->
@@ -76,5 +78,7 @@
             </geometry>
         </collision>
-        <xacro:cylinder_inertia m="0.1" r="0.05" h="0.04" />
+        <xacro:cylinder_inertia m="0.1" r="0.05" h="0.04" >
+            <origin xyz="0.0 0.0 0.0" rpy="0.0 0.0 0.0"/>
+        </xacro:cylinder_inertia>
     </link>
     <gazebo reference="left_wheel">
@@ -101,5 +105,7 @@
             </geometry>
         </collision>
-        <xacro:cylinder_inertia m="0.1" r="0.05" h="0.04" />
+        <xacro:cylinder_inertia m="0.1" r="0.05" h="0.04" >
+            <origin xyz="0.0 0.0 0.0" rpy="0.0 0.0 0.0"/>
+        </xacro:cylinder_inertia>
     </link>
     <gazebo reference="right_wheel">
@@ -125,5 +131,7 @@
             </geometry>
         </collision>
-        <xacro:sphere_inertia m="0.5" r="0.05" />
+        <xacro:sphere_inertia m="1" r="0.05" >
+            <origin xyz="0 0 0" rpy="0 0 0"/>
+        </xacro:sphere_inertia >
      </link>
      <gazebo reference="caster_wheel">
